Commit message: robot fix in world in gazebo

File: config/gazebo_SR80.urdf (robot description, URDF)
Before this commit: robot SR80, 10 links, 9 joints
Links:
- added link world
Joints:
- added joint world-base_link-fixed: type fixed, parent world, child base_link

Commit message: J2 has vel value because link mass for gazebo

File: config/gazebo_SR80.urdf (robot description, URDF)
Before this commit: robot SR80, 11 links, 10 joints
Links:
- link L1: mass 0.1 -> 0.001
- link L2: mass 0.1 -> 0.001
- link L3: mass 0.1 -> 0.001
- link L4: mass 0.1 -> 0.001
- link L5: mass 0.1 -> 0.001
- link flange: mass 0.1 -> 0.001
Joints:
- joint world-base_link-fixed: origin (none) -> xyz=0.0 0.0 0.0 rpy=0.0 0.0 0.0
